Commit message: scenes ready for RL

File: dedo/data/urdf/hanger.urdf (robot description, URDF)
Before this commit: robot rod, 3 links, 2 joints
Links:
- link rod_link_left: geometry collision cylinder length=0.15 radius=0.01; visual cylinder length=0.15 radius=0.01
- link rod_link_right: geometry collision cylinder length=0.15 radius=0.01; visual cylinder length=0.15 radius=0.01
