Commit message: preset tasks

File: dedo/data/urdf/button_fixed.urdf (robot description, URDF)
Before this commit: robot button, 3 links, 2 joints
Links:
- link button_stem: geometry collision cylinder length=0.05 radius=0.005; visual cylinder length=0.05 radius=0.005
Joints:
- joint stem_to_head: origin xyz=0 0 0.01 rpy=0 0 0 -> xyz=0 0 0.025 rpy=0 0 0
