Commit message: lasso complete

File: dedo/data/urdf/hook_small.urdf (robot description, URDF)
Before this commit: robot rod, 2 links, 1 joints
Links:
- link horizontal: geometry collision cylinder length=0.07 radius=0.01; visual cylinder length=0.07 radius=0.01
- link vertical: geometry collision cylinder length=0.02 radius=0.005; visual cylinder length=0.02 radius=0.005
