Commit message: fixing backpack's tunneling issue, not quite satistfied with the result yet

File: dedo/data/urdf/figure_headless.urdf (robot description, URDF)
Before this commit: robot mannequin, 6 links, 5 joints
Joints:
- joint left_shoulder_joint: origin xyz=0 0.1 0.27 rpy=1.57 0 0 -> xyz=0 0.08 0.27 rpy=1.57 0 0
- joint right_shoulder_joint: origin xyz=0 -0.1 0.27 rpy=1.57 0 0 -> xyz=0 -0.08 0.27 rpy=1.57 0 0

Commit message: mask

File: dedo/data/urdf/figure_headless.urdf (robot description, URDF)
Before this commit: robot mannequin, 6 links, 5 joints
Links:
- link left_arm: geometry collision cylinder length=0.1 radius=0.02; visual cylinder length=0.1 radius=0.02
- link right_arm: geometry collision cylinder length=0.1 radius=0.02; visual cylinder length=0.1 radius=0.02
Joints:
- joint left_arm_joint: origin xyz=0.05 0 -0.05 rpy=1.57 0 1.57 -> xyz=0.03 0 -0.05 rpy=1.57 0 1.57
- joint right_arm_joint: origin xyz=0.05 0 0.05 rpy=1.57 0 1.57 -> xyz=0.03 0 0.05 rpy=1.57 0 1.57

Commit message: Thinned the figure a bit, updated --max_episode_len, removed the call to debug_viz_cent_loop because these show up in RL images, updated the README

File: dedo/data/urdf/figure_headless.urdf (robot description, URDF)
Before this commit: robot mannequin, 6 links, 5 joints
Links:
- link torso: geometry collision cylinder length=0.6 radius=0.055; visual cylinder length=0.6 radius=0.055
