Commit message: bag annotation done

File: dedo/data/urdf/tallrod.urdf (robot description, URDF)
Before this commit: robot rod, 2 links, 1 joints
Links:
- link rod_link: geometry collision cylinder length=0.8 radius=0.03; visual cylinder length=0.8 radius=0.03
Joints:
- joint base_to_rod: origin xyz=0 0 0.275 rpy=0 0 0 -> xyz=0 0 0.4 rpy=0 0 0
