Commit message: procedural button

File: dedo/data/urdf/torso.urdf (robot description, URDF)
Before this commit: robot torso, 2 links, 1 joints
Links:
- link torso: geometry collision box size=3 3 4; visual box size=3 3 4
Joints:
- joint robot_to_world: origin xyz=0 0 0 rpy=0 0 0 -> xyz=1.5 -1.5 0 rpy=0 0 0
