Commit message: Small improvements to Franka

File: dedo/data/robots/franka/franka_dual.urdf (robot description, URDF)
Before this commit: robot panda, 25 links, 24 joints
Links:
- link panda_hand_l_finger_l: geometry collision mesh filename=meshes/collision/finger.stl; visual mesh filename=meshes/visual/finger_long.dae
- link panda_hand_l_finger_r: geometry collision mesh filename=meshes/collision/finger.stl; visual mesh filename=meshes/visual/finger_long.dae
- link panda_hand_r_finger_l: geometry collision mesh filename=meshes/collision/finger.stl; visual mesh filename=meshes/visual/finger_long.dae
- link panda_hand_r_finger_r: geometry collision mesh filename=meshes/collision/finger.stl; visual mesh filename=meshes/visual/finger_long.dae
Joints:
- joint robot_l_to_world: origin xyz=0.9 0 0 rpy=0 0 3.14159 -> xyz=0.9 0 0 rpy=0 0 3.141

Commit message: further fix to resolve conflicts.

File: dedo/data/robots/franka/franka_dual.urdf (robot description, URDF)
Before this commit: robot panda, 25 links, 24 joints
Links:
- link panda_hand_l_finger_l: geometry collision mesh filename=meshes/collision/finger.stl; visual mesh filename=meshes/visual/finger.dae
- link panda_hand_l_finger_r: geometry collision mesh filename=meshes/collision/finger.stl; visual mesh filename=meshes/visual/finger.dae
- link panda_hand_r_finger_l: geometry collision mesh filename=meshes/collision/finger.stl; visual mesh filename=meshes/visual/finger.dae
- link panda_hand_r_finger_r: geometry collision mesh filename=meshes/collision/finger.stl; visual mesh filename=meshes/visual/finger.dae

Commit message: Dedo robot cleanup

File: dedo/data/robots/franka/franka_dual.urdf (robot description, URDF)
Before this commit: robot panda, 25 links, 24 joints
Links:
- link panda_hand_l_finger_l: geometry collision mesh filename=meshes/collision/finger.stl; visual mesh filename=meshes/visual/finger_long_thick.dae
- link panda_hand_l_finger_r: geometry collision mesh filename=meshes/collision/finger.stl; visual mesh filename=meshes/visual/finger_long_thick.dae
- link panda_hand_r_finger_l: geometry collision mesh filename=meshes/collision/finger.stl; visual mesh filename=meshes/visual/finger_long_thick.dae
- link panda_hand_r_finger_r: geometry collision mesh filename=meshes/collision/finger.stl; visual mesh filename=meshes/visual/finger_long_thick.dae
