Commit message: robot changes

File: dedo/data/robots/fetch/fetch.urdf (robot description, URDF)
Before this commit: robot fetch, 24 links, 23 joints
Joints:
- joint torso_lift_joint: type prismatic -> fixed

Commit message: add basic support for mobile manipulator. use --robot to specify anchor/manipulators. now only fetch is tested.

File: dedo/data/robots/fetch/fetch.urdf (robot description, URDF)
Before this commit: robot fetch, 24 links, 23 joints
Joints:
- joint forearm_roll_joint: limit effort=29.35 velocity=1.571 -> lower=-1.251 upper=1.251 effort=29.35 velocity=1.571
- joint l_wheel_joint: type continuous -> fixed
- joint r_wheel_joint: type continuous -> fixed
- joint upperarm_roll_joint: limit effort=76.94 velocity=1.571 -> lower=-1.251 upper=1.251 effort=76.94 velocity=1.571
- joint wrist_roll_joint: limit effort=7.36 velocity=2.268 -> lower=-1.251 upper=1.251 effort=7.36 velocity=2.268

Commit message: Franka robot does HangGarment demo (ok, but needs tuning)

File: dedo/data/robots/fetch/fetch.urdf (robot description, URDF)
Before this commit: robot fetch, 24 links, 23 joints
Links:
- added link l_gripper_finger_link, mass 0.0798; collision mesh filename=meshes/l_gripper_finger_link.obj; visual mesh filename=meshes/l_gripper_finger_link.obj
- added link r_gripper_finger_link, mass 0.0798; collision mesh filename=meshes/r_gripper_finger_link.obj; visual mesh filename=meshes/r_gripper_finger_link.obj
Joints:
- added joint l_gripper_finger_joint: type prismatic, parent gripper_link, child l_gripper_finger_link, origin xyz=0 -0.015425 0 rpy=0 0 0, axis 0 -1 0, limit lower=0.0 upper=0.05 effort=60 velocity=0.05
- added joint r_gripper_finger_joint: type prismatic, parent gripper_link, child r_gripper_finger_link, origin xyz=0 0.015425 0 rpy=0 0 0, axis 0 1 0, limit lower=0.0 upper=0.05 effort=60 velocity=0.05
- joint eye_joint: parent head_camera_depth_frame -> head_camera_link
- joint forearm_roll_joint: limit lower=-1.251 upper=1.251 effort=29.35 velocity=1.571 -> effort=29.35 velocity=1.571
- joint head_pan_joint: type fixed -> revolute
- joint head_tilt_joint: origin xyz=0.14253 0 0.057999 rpy=0 0.17453292519943295 0 -> xyz=0.14253 0 0.057999 rpy=0 0.2617993877991494 0; type fixed -> revolute
- joint l_wheel_joint: type fixed -> continuous
- joint r_wheel_joint: type fixed -> continuous
- joint torso_lift_joint: type fixed -> prismatic
- joint upperarm_roll_joint: limit lower=-1.251 upper=1.251 effort=76.94 velocity=1.571 -> effort=76.94 velocity=1.571
- joint wrist_roll_joint: limit lower=-1.251 upper=1.251 effort=7.36 velocity=2.268 -> effort=7.36 velocity=2.268

File: dedo/data/robots/fetch/fetch_no_gripper.urdf (robot description, URDF)
Before this commit: robot fetch, 26 links, 25 joints
Links:
- removed link l_gripper_finger_link
- removed link r_gripper_finger_link
Joints:
- removed joint l_gripper_finger_joint
- removed joint r_gripper_finger_joint
- joint eye_joint: parent head_camera_link -> head_camera_depth_frame
- joint forearm_roll_joint: limit effort=29.35 velocity=1.571 -> lower=-1.251 upper=1.251 effort=29.35 velocity=1.571
- joint head_pan_joint: type revolute -> fixed
- joint head_tilt_joint: origin xyz=0.14253 0 0.057999 rpy=0 0.2617993877991494 0 -> xyz=0.14253 0 0.057999 rpy=0 0.17453292519943295 0; type revolute -> fixed
- joint l_wheel_joint: type continuous -> fixed
- joint r_wheel_joint: type continuous -> fixed
- joint torso_lift_joint: type prismatic -> fixed
- joint upperarm_roll_joint: limit effort=76.94 velocity=1.571 -> lower=-1.251 upper=1.251 effort=76.94 velocity=1.571
- joint wrist_roll_joint: limit effort=7.36 velocity=2.268 -> lower=-1.251 upper=1.251 effort=7.36 velocity=2.268

Commit message: enable base motion on fetch with 1 anchor

File: dedo/data/robots/fetch/fetch.urdf (robot description, URDF)
Before this commit: robot fetch, 26 links, 25 joints
Joints:
- joint head_pan_joint: type revolute -> fixed
- joint head_tilt_joint: type revolute -> fixed
- joint l_gripper_finger_joint: type prismatic -> fixed
- joint r_gripper_finger_joint: type prismatic -> fixed
- joint torso_lift_joint: type prismatic -> fixed

Commit message: Fixed clear_motor_control() for better reset() ; small refactoring for clipping qpos in BulletManipulator

File: dedo/data/robots/fetch/fetch.urdf (robot description, URDF)
Before this commit: robot fetch, 26 links, 25 joints
Joints:
- joint head_pan_joint: type revolute -> fixed
- joint head_tilt_joint: type revolute -> fixed
- joint l_wheel_joint: type continuous -> fixed
- joint r_wheel_joint: type continuous -> fixed
- joint torso_lift_joint: type prismatic -> fixed
